File: Lab 4 Exercise 1/Lab 4 Exercise 1.kicad_pcb (KiCad board)
At the start: 2 copper layers, 99.1 x 68.6 mm, 6 parts, among them SW1 Switch

Commit message: Lab 7 Added
Connections:
- net Net-(C1-Pad2) renamed GND
Routing:
- added copper zone on F.Cu, net GND
Changed lines of the file:
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@@
       (outputformat 1)
       (mirror false)
-      (drillshape 1)
+      (drillshape 0)
       (scaleselection 1)
       (outputdirectory "")
@@
   (net 0 "")
   (net 1 "Net-(C1-Pad1)")
-  (net 2 "Net-(C1-Pad2)")
+  (net 2 "GND")
   (net 3 "Net-(D1-Pad2)")
   (net 4 "Net-(R2-Pad1)")
@@
     (fp_line (start 3.95 -1.7) (end -1.95 -1.7) (layer "F.Fab") (width 0.1))
     (fp_line (start -1.11 -2.11) (end -2.36 -2.11) (layer "F.Fab") (width 0.1))
-    (pad "1" thru_hole roundrect (at 0 0 270) (size 1.2 1.75) (drill 0.75) (layers *.Cu *.Mask) (roundrect_rratio 0.208333)
+    (pad "1" thru_hole roundrect (at 0 0 270) (size 1.2 1.75) (drill 0.75) (layers *.Cu *.Mask) (roundrect_rratio 0.2083333333)
       (net 5 "Net-(R2-Pad2)") (pinfunction "Pin_1") (pintype "passive"))
     (pad "2" thru_hole oval (at 2 0 270) (size 1.2 1.75) (drill 0.75) (layers *.Cu *.Mask)
-      (net 2 "Net-(C1-Pad2)") (pinfunction "Pin_2") (pintype "passive"))
+      (net 2 "GND") (pinfunction "Pin_2") (pintype "passive"))
     (model "${KICAD6_3DMODEL_DIR}/Connector_JST.3dshapes/JST_PH_B2B-PH-K_1x02_P2.00mm_Vertical.wrl"
       (offset (xyz 0 0 0))
@@
     (fp_circle (center 1.27 0) (end 3.77 0) (layer "F.Fab") (width 0.1) (fill none))
     (pad "1" thru_hole rect (at 0 0 90) (size 1.8 1.8) (drill 0.9) (layers *.Cu *.Mask)
-      (net 2 "Net-(C1-Pad2)") (pinfunction "K") (pintype "passive"))
+      (net 2 "GND") (pinfunction "K") (pintype "passive"))
     (pad "2" thru_hole circle (at 2.54 0 90) (size 1.8 1.8) (drill 0.9) (layers *.Cu *.Mask)
       (net 3 "Net-(D1-Pad2)") (pinfunction "A") (pintype "passive"))
@@
       (net 1 "Net-(C1-Pad1)") (pintype "passive"))
     (pad "2" thru_hole circle (at 2 0 180) (size 1.2 1.2) (drill 0.6) (layers *.Cu *.Mask)
-      (net 2 "Net-(C1-Pad2)") (pintype "passive"))
+      (net 2 "GND") (pintype "passive"))
     (model "${KICAD6_3DMODEL_DIR}/Capacitor_THT.3dshapes/C_Radial_D5.0mm_H5.0mm_P2.00mm.wrl"
       (offset (xyz 0 0 0))
@@
   (segment (start 114.3 127.405) (end 114.66 127.765) (width 0.25) (layer "F.Cu") (net 5))
   (segment (start 114.3 73.66) (end 114.3 127.405) (width 0.25) (layer "F.Cu") (net 5))
+  (zone (net 2) (net_name "GND") (layer "F.Cu") (hatch edge 0.508)
+    (connect_pads (clearance 0.508))
+    (min_thickness 0.254) (filled_areas_thickness no)
+    (fill yes (thermal_gap 0.508) (thermal_bridge_width 0.508))
+    (polygon
+      (pts
+        (xy 200.66 132.08)
+        (xy 106.68 132.08)
+        (xy 106.68 68.58)
+        (xy 200.66 68.58)
+      )
+    )
+  )
 )
