File: Lab 4 Exercise 1/Lab 4 Exercise 1.kicad_sch (KiCad schematic)
At the start: 6 parts, among them SW1 Switch

Commit message: Lab 6 added
Parts:
- C1: footprint (none) -> Capacitor_THT:C_Radial_D5.0mm_H5.0mm_P2.00mm
- D1: footprint (none) -> LED_THT:LED_D5.0mm
- R1, R2: footprint (none) -> Resistor_THT:R_Axial_DIN0516_L15.5mm_D5.0mm_P20.32mm_Horizontal
- SW1: footprint (none) -> Button_Switch_THT:SW_E-Switch_EG1224_SPDT_Angled
- V1: footprint (none) -> Connector_JST:JST_PH_B2B-PH-K_1x02_P2.00mm_Vertical
Connections:
- net at R2.2: now also V1.1 (Pin_1)
Other:
- moved on the sheet: V1
Changed lines of the file:
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@@
   (junction (at 91.44 44.45) (diameter 0) (color 0 0 0 0)
   )
+  (junction (at 107.95 85.09) (diameter 0) (color 0 0 0 0)
+  )
   (junction (at 107.95 46.99) (diameter 0) (color 0 0 0 0)
-  )
-  (junction (at 107.95 85.09) (diameter 0) (color 0 0 0 0)
   )
   (wire (pts (xy 91.44 44.45) (xy 93.98 44.45))
     (stroke (width 0) (type default) (color 0 0 0 0))
   )
-  (wire (pts (xy 107.95 85.09) (xy 91.44 85.09))
+  (wire (pts (xy 90.17 82.55) (xy 99.06 82.55))
     (stroke (width 0) (type default) (color 0 0 0 0))
   )
@@
     (stroke (width 0) (type default) (color 0 0 0 0))
   )
-  (wire (pts (xy 71.12 82.55) (xy 86.36 82.55))
+  (wire (pts (xy 99.06 85.09) (xy 107.95 85.09))
+    (stroke (width 0) (type default) (color 0 0 0 0))
+  )
+  (wire (pts (xy 71.12 82.55) (xy 87.63 82.55))
     (stroke (width 0) (type default) (color 0 0 0 0))
   )
@@
   )
   (wire (pts (xy 101.6 46.99) (xy 107.95 46.99))
+    (stroke (width 0) (type default) (color 0 0 0 0))
+  )
+  (wire (pts (xy 99.06 82.55) (xy 99.06 85.09))
     (stroke (width 0) (type default) (color 0 0 0 0))
   )
@@
       (effects (font (size 1.27 1.27)) (justify left))
     )
-    (property "Footprint" "" (id 2) (at 69.342 58.42 90)
+    (property "Footprint" "Resistor_THT:R_Axial_DIN0516_L15.5mm_D5.0mm_P20.32mm_Horizontal" (id 2) (at 69.342 58.42 90)
       (effects (font (size 1.27 1.27)) hide)
     )
@@
     (pin "2")
   )
-  (symbol (lib_id "Connector:Conn_01x02_Male") (at 86.36 82.55 0) (unit 1)
+  (symbol (lib_id "Connector:Conn_01x02_Male") (at 87.63 87.63 90) (unit 1)
     (in_bom yes) (on_board yes) (fields_autoplaced)
-    (property "Reference" "V1" (id 0) (at 86.995 77.47 0))
-    (property "Value" "9V" (id 1) (at 86.995 80.01 0))
-    (property "Footprint" "" (id 2) (at 86.36 82.55 0)
+    (property "Reference" "V1" (id 0) (at 91.44 85.7249 90)
+      (effects (font (size 1.27 1.27)) (justify right))
+    )
+    (property "Value" "9V" (id 1) (at 91.44 88.2649 90)
+      (effects (font (size 1.27 1.27)) (justify right))
+    )
+    (property "Footprint" "Connector_JST:JST_PH_B2B-PH-K_1x02_P2.00mm_Vertical" (id 2) (at 87.63 87.63 0)
       (effects (font (size 1.27 1.27)) hide)
     )
-    (property "Datasheet" "~" (id 3) (at 86.36 82.55 0)
+    (property "Datasheet" "~" (id 3) (at 87.63 87.63 0)
       (effects (font (size 1.27 1.27)) hide)
     )
@@
       (effects (font (size 1.27 1.27)) (justify right))
     )
-    (property "Footprint" "" (id 2) (at 139.7 71.12 0)
+    (property "Footprint" "LED_THT:LED_D5.0mm" (id 2) (at 139.7 71.12 0)
       (effects (font (size 1.27 1.27)) hide)
     )
@@
       (effects (font (size 1.27 1.27)) (justify left))
     )
-    (property "Footprint" "" (id 2) (at 137.922 53.34 90)
+    (property "Footprint" "Resistor_THT:R_Axial_DIN0516_L15.5mm_D5.0mm_P20.32mm_Horizontal" (id 2) (at 137.922 53.34 90)
       (effects (font (size 1.27 1.27)) hide)
     )
@@
     (property "Reference" "SW1" (id 0) (at 96.52 36.83 0))
     (property "Value" "Switch" (id 1) (at 96.52 39.37 0))
-    (property "Footprint" "" (id 2) (at 96.52 44.45 0)
+    (property "Footprint" "Button_Switch_THT:SW_E-Switch_EG1224_SPDT_Angled" (id 2) (at 96.52 44.45 0)
       (effects (font (size 1.27 1.27)) hide)
     )
@@
       (effects (font (size 1.27 1.27)) (justify left))
     )
-    (property "Footprint" "" (id 2) (at 108.9152 60.96 0)
+    (property "Footprint" "Capacitor_THT:C_Radial_D5.0mm_H5.0mm_P2.00mm" (id 2) (at 108.9152 60.96 0)
       (effects (font (size 1.27 1.27)) hide)
     )
@@
   (symbol_instances
     (path "/bbcaf60c-8637-4c94-986e-92f7c9b2c30a"
-      (reference "C1") (unit 1) (value "4.7 mu F") (footprint "")
+      (reference "C1") (unit 1) (value "4.7 mu F") (footprint "Capacitor_THT:C_Radial_D5.0mm_H5.0mm_P2.00mm")
     )
     (path "/3dd61fe4-9464-477e-bec3-0b4b2e272e4f"
-      (reference "D1") (unit 1) (value "LED") (footprint "")
+      (reference "D1") (unit 1) (value "LED") (footprint "LED_THT:LED_D5.0mm")
     )
     (path "/74b9a99f-4f90-4148-bbcc-c4f6dda196eb"
-      (reference "R1") (unit 1) (value "20K") (footprint "")
+      (reference "R1") (unit 1) (value "20K") (footprint "Resistor_THT:R_Axial_DIN0516_L15.5mm_D5.0mm_P20.32mm_Horizontal")
     )
     (path "/13d3796c-6914-4d1e-95a7-6bb03ad60c3f"
-      (reference "R2") (unit 1) (value "2.2K") (footprint "")
+      (reference "R2") (unit 1) (value "2.2K") (footprint "Resistor_THT:R_Axial_DIN0516_L15.5mm_D5.0mm_P20.32mm_Horizontal")
     )
     (path "/8733ca4b-faf0-46e5-8e1d-9bb54a9ce88b"
-      (reference "SW1") (unit 1) (value "Switch") (footprint "")
+      (reference "SW1") (unit 1) (value "Switch") (footprint "Button_Switch_THT:SW_E-Switch_EG1224_SPDT_Angled")
     )
     (path "/3bbf349b-9396-43f5-9549-efcf4a16702c"
-      (reference "V1") (unit 1) (value "9V") (footprint "")
+      (reference "V1") (unit 1) (value "9V") (footprint "Connector_JST:JST_PH_B2B-PH-K_1x02_P2.00mm_Vertical")
     )
   )

Commit message: Lab 7 Added
Connections:
- net GND: now reaches C1.2, D1.1 (K), V1.2 (Pin_2)
Changed lines of the file:
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@@
     (pin "3")
+  )
+  (symbol (lib_id "power:GND") (at 107.95 85.09 0) (unit 1)
+    (in_bom yes) (on_board yes) (fields_autoplaced)
+    (property "Reference" "#PWR0101" (id 0) (at 107.95 91.44 0)
+      (effects (font (size 1.27 1.27)) hide)
+    )
+    (property "Value" "GND" (id 1) (at 107.95 90.17 0))
+    (property "Footprint" "" (id 2) (at 107.95 85.09 0)
+      (effects (font (size 1.27 1.27)) hide)
+    )
+    (property "Datasheet" "" (id 3) (at 107.95 85.09 0)
+      (effects (font (size 1.27 1.27)) hide)
+    )
+    (pin "1")
   )
   (symbol (lib_id "Device:C_Polarized") (at 107.95 57.15 0) (unit 1)
@@
   )
   (symbol_instances
+    (path "/b94fadd7-c1e7-4fa7-b75f-db21dbfef302"
+      (reference "#PWR0101") (unit 1) (value "GND") (footprint "")
+    )
     (path "/bbcaf60c-8637-4c94-986e-92f7c9b2c30a"
       (reference "C1") (unit 1) (value "4.7 mu F") (footprint "Capacitor_THT:C_Radial_D5.0mm_H5.0mm_P2.00mm")
