File: Lab 4 Exercise 1/Lab 4 Exercise 2/Lab 4 Exercise 2.kicad_pcb (KiCad board)
At the start: 2 copper layers, 58.4 x 43.2 mm, 10 parts, among them J1 , U1 NE555D

Commit message: Lab 8 Added
Routing:
- net /pin_2: track 31.8 -> 26.7 mm
- net +9V: track 46.8 -> 48.7 mm, vias 2 -> 3
- added copper zone on F.Cu, net GND
Changed lines of the file:
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@@
       (outputformat 1)
       (mirror false)
-      (drillshape 1)
+      (drillshape 0)
       (scaleselection 1)
       (outputdirectory "")
@@
     (fp_line (start 1 0.625) (end -1 0.625) (layer "F.Fab") (width 0.1))
     (fp_line (start -1 -0.625) (end 1 -0.625) (layer "F.Fab") (width 0.1))
-    (pad "1" smd roundrect (at -1.0375 0 90) (size 1.175 1.45) (layers "F.Cu" "F.Paste" "F.Mask") (roundrect_rratio 0.212766)
+    (pad "1" smd roundrect (at -1.0375 0 90) (size 1.175 1.45) (layers "F.Cu" "F.Paste" "F.Mask") (roundrect_rratio 0.2127659574)
       (net 3 "Net-(C2-Pad1)") (pintype "passive"))
-    (pad "2" smd roundrect (at 1.0375 0 90) (size 1.175 1.45) (layers "F.Cu" "F.Paste" "F.Mask") (roundrect_rratio 0.212766)
+    (pad "2" smd roundrect (at 1.0375 0 90) (size 1.175 1.45) (layers "F.Cu" "F.Paste" "F.Mask") (roundrect_rratio 0.2127659574)
       (net 2 "GND") (pintype "passive"))
     (model "${KICAD6_3DMODEL_DIR}/Capacitor_SMD.3dshapes/C_0805_2012Metric.wrl"
@@
     (fp_line (start -1 -0.625) (end 1 -0.625) (layer "F.Fab") (width 0.1))
     (fp_line (start 1 -0.625) (end 1 0.625) (layer "F.Fab") (width 0.1))
-    (pad "1" smd roundrect (at -1 0 180) (size 1.2 1.4) (layers "F.Cu" "F.Paste" "F.Mask") (roundrect_rratio 0.208333)
+    (pad "1" smd roundrect (at -1 0 180) (size 1.2 1.4) (layers "F.Cu" "F.Paste" "F.Mask") (roundrect_rratio 0.2083333333)
       (net 7 "Net-(R1-Pad2)") (pintype "passive"))
-    (pad "2" smd roundrect (at 1 0 180) (size 1.2 1.4) (layers "F.Cu" "F.Paste" "F.Mask") (roundrect_rratio 0.208333)
+    (pad "2" smd roundrect (at 1 0 180) (size 1.2 1.4) (layers "F.Cu" "F.Paste" "F.Mask") (roundrect_rratio 0.2083333333)
       (net 1 "Net-(C1-Pad1)") (pintype "passive"))
     (model "${KICAD6_3DMODEL_DIR}/Resistor_SMD.3dshapes/R_0805_2012Metric.wrl"
@@
     (fp_line (start -1.2 -0.8) (end -1.6 -0.4) (layer "F.Fab") (width 0.1))
     (fp_line (start -1.6 0.8) (end 1.6 0.8) (layer "F.Fab") (width 0.1))
-    (pad "1" smd roundrect (at -1.4375 0 90) (size 1.575 1.35) (layers "F.Cu" "F.Paste" "F.Mask") (roundrect_rratio 0.185185)
+    (pad "1" smd roundrect (at -1.4375 0 90) (size 1.575 1.35) (layers "F.Cu" "F.Paste" "F.Mask") (roundrect_rratio 0.1851851852)
       (net 1 "Net-(C1-Pad1)") (pintype "passive"))
-    (pad "2" smd roundrect (at 1.4375 0 90) (size 1.575 1.35) (layers "F.Cu" "F.Paste" "F.Mask") (roundrect_rratio 0.185185)
+    (pad "2" smd roundrect (at 1.4375 0 90) (size 1.575 1.35) (layers "F.Cu" "F.Paste" "F.Mask") (roundrect_rratio 0.1851851852)
       (net 2 "GND") (pintype "passive"))
     (model "${KICAD6_3DMODEL_DIR}/Capacitor_Tantalum_SMD.3dshapes/CP_EIA-3216-18_Kemet-A.wrl"
@@
     (fp_line (start -1 0.625) (end -1 -0.625) (layer "F.Fab") (width 0.1))
     (fp_line (start 1 0.625) (end -1 0.625) (layer "F.Fab") (width 0.1))
-    (pad "1" smd roundrect (at -1 0 270) (size 1.2 1.4) (layers "F.Cu" "F.Paste" "F.Mask") (roundrect_rratio 0.208333)
+    (pad "1" smd roundrect (at -1 0 270) (size 1.2 1.4) (layers "F.Cu" "F.Paste" "F.Mask") (roundrect_rratio 0.2083333333)
       (net 5 "+9V") (pintype "passive"))
-    (pad "2" smd roundrect (at 1 0 270) (size 1.2 1.4) (layers "F.Cu" "F.Paste" "F.Mask") (roundrect_rratio 0.208333)
+    (pad "2" smd roundrect (at 1 0 270) (size 1.2 1.4) (layers "F.Cu" "F.Paste" "F.Mask") (roundrect_rratio 0.2083333333)
       (net 7 "Net-(R1-Pad2)") (pintype "passive"))
     (model "${KICAD6_3DMODEL_DIR}/Resistor_SMD.3dshapes/R_0805_2012Metric.wrl"
@@
     (fp_line (start 1 -0.625) (end 1 0.625) (layer "F.Fab") (width 0.1))
     (fp_line (start -1 0.625) (end -1 -0.625) (layer "F.Fab") (width 0.1))
-    (pad "1" smd roundrect (at -1 0 180) (size 1.2 1.4) (layers "F.Cu" "F.Paste" "F.Mask") (roundrect_rratio 0.208333)
+    (pad "1" smd roundrect (at -1 0 180) (size 1.2 1.4) (layers "F.Cu" "F.Paste" "F.Mask") (roundrect_rratio 0.2083333333)
       (net 4 "Net-(D1-Pad1)") (pintype "passive"))
-    (pad "2" smd roundrect (at 1 0 180) (size 1.2 1.4) (layers "F.Cu" "F.Paste" "F.Mask") (roundrect_rratio 0.208333)
+    (pad "2" smd roundrect (at 1 0 180) (size 1.2 1.4) (layers "F.Cu" "F.Paste" "F.Mask") (roundrect_rratio 0.2083333333)
       (net 8 "/pin_3") (pintype "passive"))
     (model "${KICAD6_3DMODEL_DIR}/Resistor_SMD.3dshapes/R_0805_2012Metric.wrl"
@@
     (fp_line (start -1.6 0.8) (end 1.6 0.8) (layer "F.Fab") (width 0.1))
     (fp_line (start 1.6 0.8) (end 1.6 -0.8) (layer "F.Fab") (width 0.1))
-    (pad "1" smd roundrect (at -1.4875 0 270) (size 1.425 1.75) (layers "F.Cu" "F.Paste" "F.Mask") (roundrect_rratio 0.175439)
+    (pad "1" smd roundrect (at -1.4875 0 270) (size 1.425 1.75) (layers "F.Cu" "F.Paste" "F.Mask") (roundrect_rratio 0.1754392982)
       (net 2 "GND") (pinfunction "K") (pintype "passive"))
-    (pad "2" smd roundrect (at 1.4875 0 270) (size 1.425 1.75) (layers "F.Cu" "F.Paste" "F.Mask") (roundrect_rratio 0.175439)
+    (pad "2" smd roundrect (at 1.4875 0 270) (size 1.425 1.75) (layers "F.Cu" "F.Paste" "F.Mask") (roundrect_rratio 0.1754392982)
       (net 6 "Net-(D2-Pad2)") (pinfunction "A") (pintype "passive"))
     (model "${KICAD6_3DMODEL_DIR}/LED_SMD.3dshapes/LED_1206_3216Metric.wrl"
@@
     (fp_line (start -1.6 -0.4) (end -1.6 0.8) (layer "F.Fab") (width 0.1))
     (fp_line (start 1.6 -0.8) (end -1.2 -0.8) (layer "F.Fab") (width 0.1))
-    (pad "1" smd roundrect (at -1.4875 0) (size 1.425 1.75) (layers "F.Cu" "F.Paste" "F.Mask") (roundrect_rratio 0.175439)
+    (pad "1" smd roundrect (at -1.4875 0) (size 1.425 1.75) (layers "F.Cu" "F.Paste" "F.Mask") (roundrect_rratio 0.1754392982)
       (net 4 "Net-(D1-Pad1)") (pinfunction "K") (pintype "passive"))
-    (pad "2" smd roundrect (at 1.4875 0) (size 1.425 1.75) (layers "F.Cu" "F.Paste" "F.Mask") (roundrect_rratio 0.175439)
+    (pad "2" smd roundrect (at 1.4875 0) (size 1.425 1.75) (layers "F.Cu" "F.Paste" "F.Mask") (roundrect_rratio 0.1754392982)
       (net 5 "+9V") (pinfunction "A") (pintype "passive"))
     (model "${KICAD6_3DMODEL_DIR}/LED_SMD.3dshapes/LED_1206_3216Metric.wrl"
@@
     (fp_line (start 1 -0.625) (end 1 0.625) (layer "F.Fab") (width 0.1))
     (fp_line (start -1 -0.625) (end 1 -0.625) (layer "F.Fab") (width 0.1))
-    (pad "1" smd roundrect (at -1 0 180) (size 1.2 1.4) (layers "F.Cu" "F.Paste" "F.Mask") (roundrect_rratio 0.208333)
+    (pad "1" smd roundrect (at -1 0 180) (size 1.2 1.4) (layers "F.Cu" "F.Paste" "F.Mask") (roundrect_rratio 0.2083333333)
       (net 8 "/pin_3") (pintype "passive"))
-    (pad "2" smd roundrect (at 1 0 180) (size 1.2 1.4) (layers "F.Cu" "F.Paste" "F.Mask") (roundrect_rratio 0.208333)
+    (pad "2" smd roundrect (at 1 0 180) (size 1.2 1.4) (layers "F.Cu" "F.Paste" "F.Mask") (roundrect_rratio 0.2083333333)
       (net 6 "Net-(D2-Pad2)") (pintype "passive"))
     (model "${KICAD6_3DMODEL_DIR}/Resistor_SMD.3dshapes/R_0805_2012Metric.wrl"
@@
   (gr_rect (start 124.46 78.74) (end 182.88 121.92) (layer "Edge.Cuts") (width 0.1) (fill none))
   (gr_circle (center 177.8 83.82) (end 180.34 83.82) (layer "Edge.Cuts") (width 0.1) (fill none))
-  (gr_text "EE 201" (at 177.8 116.84) (layer "Edge.Cuts")
+  (gr_text "EE 201" (at 177.8 116.84) (layer "F.SilkS")
     (effects (font (size 1 1) (thickness 0.15)))
   )
-  (gr_text "Arya Goel" (at 177.8 119.38) (layer "Edge.Cuts")
+  (gr_text "Arya Goel" (at 177.8 119.38) (layer "F.SilkS")
     (effects (font (size 1 1) (thickness 0.15)))
   )
@@
   (segment (start 152.4 97.09) (end 152.335 97.155) (width 0.25) (layer "F.Cu") (net 5))
   (segment (start 152.97 96.52) (end 154.94 96.52) (width 0.25) (layer "F.Cu") (net 5))
-  (segment (start 147.385 107.7975) (end 148.8075 109.22) (width 0.25) (layer "F.Cu") (net 5))
-  (segment (start 147.385 100.965) (end 147.385 107.7975) (width 0.25) (layer "F.Cu") (net 5))
   (segment (start 154.94 108.22) (end 153.94 109.22) (width 0.25) (layer "F.Cu") (net 5))
   (segment (start 146.75 101.6) (end 147.385 100.965) (width 0.25) (layer "F.Cu") (net 5))
@@
   (via (at 154.94 96.52) (size 0.8) (drill 0.4) (layers "F.Cu" "B.Cu") (net 5))
   (via (at 144.78 101.6) (size 0.8) (drill 0.4) (layers "F.Cu" "B.Cu") (net 5))
+  (via (at 152.4 109.22) (size 0.8) (drill 0.4) (layers "F.Cu" "B.Cu") (net 5))
   (segment (start 147.32 99.06) (end 144.78 101.6) (width 0.25) (layer "B.Cu") (net 5))
   (segment (start 152.4 99.06) (end 147.32 99.06) (width 0.25) (layer "B.Cu") (net 5))
+  (segment (start 144.78 101.6) (end 152.4 109.22) (width 0.25) (layer "B.Cu") (net 5))
   (segment (start 154.94 96.52) (end 152.4 99.06) (width 0.25) (layer "B.Cu") (net 5))
   (segment (start 138.2125 100.5475) (end 137.687064 101.072936) (width 0.25) (layer "F.Cu") (net 6))
@@
   (via (at 157.48 99.06) (size 0.8) (drill 0.4) (layers "F.Cu" "B.Cu") (net 9))
   (via (at 144.78 99.06) (size 0.8) (drill 0.4) (layers "F.Cu" "B.Cu") (net 9))
-  (segment (start 142.24 104.14) (end 142.24 101.6) (width 0.25) (layer "B.Cu") (net 9))
-  (segment (start 152.4 104.14) (end 142.24 104.14) (width 0.25) (layer "B.Cu") (net 9))
-  (segment (start 157.48 99.06) (end 152.4 104.14) (width 0.25) (layer "B.Cu") (net 9))
-  (segment (start 142.24 101.6) (end 144.78 99.06) (width 0.25) (layer "B.Cu") (net 9))
+  (segment (start 157.48 96.52) (end 157.48 99.06) (width 0.25) (layer "B.Cu") (net 9))
+  (segment (start 144.78 99.06) (end 149.86 93.98) (width 0.25) (layer "B.Cu") (net 9))
+  (segment (start 154.94 93.98) (end 157.48 96.52) (width 0.25) (layer "B.Cu") (net 9))
+  (segment (start 149.86 93.98) (end 154.94 93.98) (width 0.25) (layer "B.Cu") (net 9))
+  (zone (net 2) (net_name "GND") (layer "F.Cu") (hatch edge 0.508)
+    (connect_pads (clearance 0.508))
+    (min_thickness 0.254) (filled_areas_thickness no)
+    (fill yes (thermal_gap 0.508) (thermal_bridge_width 0.508))
+    (polygon
+      (pts
+        (xy 180.34 119.38)
+        (xy 127 119.38)
+        (xy 127 81.28)
+        (xy 180.34 81.28)
+      )
+    )
+  )
 )
